Commit message: update

File: simulation/autolabor_description/urdf/autolabor_pro1_sim.urdf (robot description, URDF)
Before this commit: robot autolabor_description, 2 links, 1 joints
Links:
- removed link model_link
- added link world
- link base_link: mass None -> 10; geometry collision mesh filename=package://autolabor_description/meshes/autolabor_pro1.stl scale=0.001 0.001 0.001; visual mesh filename=package://autolabor_description/meshes/untitled.dae scale=0.001 0.001 0.001
Joints:
- removed joint model_to_base
- added joint joint1: type continuous, parent world, child base_link, origin xyz=0 0 0 rpy=0 0 0

Commit message: update

File: simulation/autolabor_description/urdf/autolabor_pro1_sim.urdf (robot description, URDF)
Before this commit: robot autolabor_description, 2 links, 1 joints
Links:
- link base_link: geometry collision mesh filename=package://autolabor_description/meshes/autolabor_pro1.stl scale=0.001 0.001 0.001; visual mesh filename=package://autolabor_description/meshes/autolabor_pro1.stl scale=0.001 0.001 0.001

Commit message: update

File: simulation/autolabor_description/urdf/autolabor_pro1_sim.urdf (robot description, URDF)
Before this commit: robot autolabor_description, 2 links, 1 joints
Links:
- added link back_link, mass 1; collision mesh filename=package://autolabor_description/meshes/backwheel.stl; visual mesh filename=package://autolabor_description/meshes/backwheel.stl
- added link front_link, mass 1; collision mesh filename=package://autolabor_description/meshes/frontwheel.stl; visual mesh filename=package://autolabor_description/meshes/frontwheel.stl
- link base_link: geometry collision mesh filename=package://autolabor_description/meshes/body.stl; visual mesh filename=package://autolabor_description/meshes/body.stl
Joints:
- added joint fixed_joint: type fixed, parent world, child base_link, origin xyz=0 0 0 rpy=0 0 0
- added joint joint2: type revolute, parent base_link, child back_link, origin xyz=0 0 0 rpy=0 0 0, axis 1 0 0, limit lower=-1.57 upper=0 effort=1 velocity=10
- joint joint1: axis (none) -> 1 0 0; child base_link -> front_link; limit (none) -> lower=-1.57 upper=0 effort=1 velocity=10; parent world -> base_link; type continuous -> revolute

Commit message: update

File: simulation/autolabor_description/urdf/autolabor_pro1_sim.urdf (robot description, URDF)
Before this commit: robot autolabor_description, 4 links, 3 joints
Joints:
- joint joint1: limit lower=-1.57 upper=0 effort=1 velocity=10 -> lower=-1.79769e+308 upper=1.79769e+308 effort=10 velocity=10
- joint joint2: limit lower=-1.57 upper=0 effort=1 velocity=10 -> lower=-1.79769e+308 upper=1.79769e+308 effort=10 velocity=10

File: simulation/autolabor_description/urdf/autolabor_pro1_sim_2_cam.urdf (robot description, URDF)
Before this commit: robot autolabor_description, 6 links, 5 joints
Links:
- added link camera, mass 0.001; collision box size=0.1 0.1 0.1; visual box size=0.1 0.1 0.1
Joints:
- added joint cam_joint: type fixed, parent base_link, child camera, origin xyz=0 0.8 1 rpy=0 1.5707 0
- joint bljoint: axis -1  0  0 -> (none); limit lower=-1.79769e+308 upper=1.79769e+308 effort=10 velocity=10 -> (none); origin xyz=0.2827356159687042 0.2670927047729492 -0.03086165525019169 rpy=0  0  3.14159 -> xyz=0.2827356159687042 0.2670927047729492 -0.03086165525019169 rpy=0  0  0; type revolute -> fixed
- joint brjoint: axis 1  0  0 -> (none); limit lower=-1.79769e+308 upper=1.79769e+308 effort=10 velocity=10 -> (none); type revolute -> fixed
- joint fljoint: axis -1  0  0 -> 1  0  0; origin xyz=0.2827356159687042 -0.1203216165304184 -0.02870248258113861 rpy=0  0  3.14159 -> xyz=0.2827356159687042 -0.1203216165304184 -0.02870248258113861 rpy=0  0  0
