Commit message: update

File: simulation/autolabor_description/urdf/autolabor_pro1_sim_2.urdf (robot description, URDF)
Before this commit: robot autolabor_description, 6 links, 5 joints
Links:
- removed link back_left_link
- removed link back_right_link
- removed link front_left_link
- removed link front_right_link
- removed link world
- added link back_left_wheel, mass 1; collision mesh filename=package://autolabor_description/meshes/wheel.stl scale=1 1 1; visual mesh filename=package://autolabor_description/meshes/wheel.stl scale=1 1 1
- added link back_right_wheel, mass 1; collision mesh filename=package://autolabor_description/meshes/wheel.stl scale=1 1 1; visual mesh filename=package://autolabor_description/meshes/wheel.stl scale=1 1 1
- added link front_left_wheel, mass 1; collision mesh filename=package://autolabor_description/meshes/wheel.stl scale=1 1 1; visual mesh filename=package://autolabor_description/meshes/wheel.stl scale=1 1 1
- added link front_right_wheel, mass 1; collision mesh filename=package://autolabor_description/meshes/wheel.stl scale=1 1 1; visual mesh filename=package://autolabor_description/meshes/wheel.stl scale=1 1 1
- added link odom
- link base_link: geometry collision mesh filename=package://autolabor_description/meshes/body.stl scale=1 1 1; visual mesh filename=package://autolabor_description/meshes/body.stl scale=1 1 1
Joints:
- removed joint fixed_joint
- added joint dummy_joint: type fixed, parent odom, child base_link, origin xyz=0 0 0 rpy=0 0 0
- joint bljoint: axis 1 0 0 -> -1  0  0; child back_left_link -> back_left_wheel; limit lower=-1.57 upper=0 effort=1 velocity=10 -> lower=-1.79769e+308 upper=1.79769e+308 effort=10 velocity=10; origin xyz=0.27769 0.19609 0.02618 rpy=0 0 3.14159 -> xyz=0.2827356159687042 0.2670927047729492 -0.03086165525019169 rpy=0  0  3.14159
- joint brjoint: axis 1 0 0 -> 1  0  0; child back_right_link -> back_right_wheel; limit lower=-1.57 upper=0 effort=1 velocity=10 -> lower=-1.79769e+308 upper=1.79769e+308 effort=10 velocity=10; origin xyz=-0.27769 0.19609 0.02618 rpy=0 0 0 -> xyz=-0.2786993682384491 0.2670927047729492 -0.03011767752468586 rpy=0  0  0
- joint fljoint: axis 1 0 0 -> 0  0  1; child front_left_link -> front_left_wheel; limit lower=-1.57 upper=0 effort=1 velocity=10 -> lower=-0.3 upper=0.3 effort=10 velocity=10; origin xyz=0.27769 -0.1894 0.02618 rpy=0 0 3.14159 -> xyz=0.2827356159687042 -0.1203216165304184 -0.02870248258113861 rpy=0  0  3.14159
- joint frjoint: axis 1 0 0 -> 0  0  1; child front_right_link -> front_right_wheel; limit lower=-1.57 upper=0 effort=1 velocity=10 -> lower=-0.3 upper=0.3 effort=10 velocity=10; origin xyz=-0.27769 -0.1894 0.02618 rpy=0 0 0 -> xyz=-0.2786993682384491 -0.12106603384017944 -0.02870245650410652 rpy=0  0  0

Commit message: update

File: simulation/autolabor_description/urdf/autolabor_pro1_sim_2.urdf (robot description, URDF)
Before this commit: robot autolabor_description, 6 links, 5 joints
Joints:
- joint bljoint: axis -1  0  0 -> 1  0  0; origin xyz=0.2827356159687042 0.2670927047729492 -0.03086165525019169 rpy=0  0  3.14159 -> xyz=0.2827356159687042 0.2670927047729492 -0.02870245650410652 rpy=0  0  0
- joint brjoint: origin xyz=-0.2786993682384491 0.2670927047729492 -0.03011767752468586 rpy=0  0  0 -> xyz=-0.2786993682384491 0.2670927047729492 -0.02870245650410652 rpy=0  0  0
- joint fljoint: axis -1  0  0 -> 1  0  0; origin xyz=0.2827356159687042 -0.1203216165304184 -0.02870248258113861 rpy=0  0  3.14159 -> xyz=0.2827356159687042 -0.1203216165304184 -0.02870248258113861 rpy=0  0  0

File: simulation/autolabor_description/urdf/model.urdf (robot description, URDF)
Before this commit: robot autolabor_description, 7 links, 6 joints
Joints:
- joint bljoint: axis 0  0 1 -> 0 0 1
- joint brjoint: axis 0  0 1 -> 0 0 1
- joint fljoint: axis 0  0 1 -> 0 0 1
- joint frjoint: axis 0  0 1 -> 0 0 1
