Commit message: update

File: simulation/autolabor_description/urdf/model.urdf (robot description, URDF)
Before this commit: robot autolabor_description, 7 links, 6 joints
Links:
- removed link odom
- added link body, mass 1.0; collision box size=0.7 0.4 0.16; visual box size=0.7 0.4 0.16
- added link ray, mass 0.001; collision box size=0.1 0.1 0.1; visual box size=0.1 0.1 0.1
- link base_link: mass 1.0 -> None; geometry 
Joints:
- added joint ray_joint: type fixed, parent body, child ray, origin xyz=0.8 0 1.0 rpy=0 0 0
- joint bljoint: origin xyz=-0.23 -0.22 0 rpy=3.14159 -1.57079  3.14159 -> xyz=-0.22 0.23 0 rpy=-1.57079 0  0; parent base_link -> body
- joint brjoint: origin xyz=0.23 -0.22 0 rpy=3.14159 -1.57079  3.14159 -> xyz=-0.22 -0.23 0 rpy=-1.57079 0  0; parent base_link -> body
- joint cam_joint: origin xyz=0 0.8 0.5 rpy=0 1.5707 0 -> xyz=0.8 0 0.5 rpy=0 1.5707 0; parent base_link -> body
- joint dummy_joint: child base_link -> body; parent odom -> base_link
- joint fljoint: limit lower=-1.79769e+308 upper=1.79769e+308 effort=10 velocity=10 -> (none); origin xyz=-0.23  0.22 0 rpy=3.14159 -1.57079  3.14159 -> xyz=0.22  0.23 0 rpy=-1.57079 0  0; parent base_link -> body; type revolute -> continuous
- joint frjoint: limit lower=-1.79769e+308 upper=1.79769e+308 effort=10 velocity=10 -> (none); origin xyz=0.23  0.22 0 rpy=3.14159 -1.57079  3.14159 -> xyz=0.22  -0.23 0 rpy=-1.57079 0  00; parent base_link -> body; type revolute -> continuous

Commit message: update

File: simulation/autolabor_description/urdf/model.urdf (robot description, URDF)
Before this commit: robot autolabor_description, 8 links, 7 joints
Links:
- link blw: mass 0.8 -> 1.0
- link body: mass 1 -> 2
- link brw: mass 0.8 -> 1.0
- link flw: mass 0.8 -> 1.0
- link frw: mass 0.8 -> 1.0
Joints:
- joint bljoint: limit lower=-1.79769e+308 upper=1.79769e+308 effort=50 velocity=50 -> lower=-1.79769e+308 upper=1.79769e+308 effort=100 velocity=50
- joint brjoint: limit lower=-1.79769e+308 upper=1.79769e+308 effort=50 velocity=50 -> lower=-1.79769e+308 upper=1.79769e+308 effort=100 velocity=50
- joint fljoint: limit lower=-1.79769e+308 upper=1.79769e+308 effort=50 velocity=50 -> lower=-1.79769e+308 upper=1.79769e+308 effort=100 velocity=50
- joint frjoint: limit lower=-1.79769e+308 upper=1.79769e+308 effort=50 velocity=50 -> lower=-1.79769e+308 upper=1.79769e+308 effort=100 velocity=50; origin xyz=0.22  -0.225 0 rpy=-1.570796327 0  00 -> xyz=0.22  -0.225 0 rpy=-1.570796327 0  0
